File: KiCAD/K68-CPUB.kicad_sch (KiCad schematic)
At the start: 64 parts, among them J1 PIA Con, J2 SBC68 BUS, J3 SERIAL COn, J4 Barrel_Jack_Switch, SW1 SW_SPDT, SW2 BOARD SW, SW3 ECHO SW, U1 74LS123, U10 74LS244, U11 74LS244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

Commit message: ビアのテンティングを変更してREV2ガーバー再出力
Changed lines of the file:
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@@
 (kicad_sch
-	(version 20231120)
+	(version 20250114)
 	(generator "eeschema")
-	(generator_version "8.0")
+	(generator_version "9.0")
 	(paper "A3")
 	(title_block
@@
 		(company "KUNI-NET")
 	)
+	(text "RxD"
+		(exclude_from_sim no)
+		(at 359.41 135.89 0)
+		(effects
+			(font
+				(size 1.27 1.27)
+			)
+			(justify left bottom)
+		)
+	)
+	(text "+5V"
+		(exclude_from_sim no)
+		(at 359.41 130.81 0)
+		(effects
+			(font
+				(size 1.27 1.27)
+			)
+			(justify left bottom)
+		)
+	)
+	(text "GND"
+		(exclude_from_sim no)
+		(at 359.41 125.73 0)
+		(effects
+			(font
+				(size 1.27 1.27)
+			)
+			(justify left bottom)
+		)
+	)
+	(text "TxD"
+		(exclude_from_sim no)
+		(at 359.41 133.35 0)
+		(effects
+			(font
+				(size 1.27 1.27)
+			)
+			(justify left bottom)
+		)
+	)
+	(text "CTS"
+		(exclude_from_sim no)
+		(at 359.41 128.27 0)
+		(effects
+			(font
+				(size 1.27 1.27)
+			)
+			(justify left bottom)
+		)
+	)
+	(text "RTS"
+		(exclude_from_sim no)
+		(at 359.41 138.43 0)
+		(effects
+			(font
+				(size 1.27 1.27)
+			)
+			(justify left bottom)
+		)
+	)
 	(junction
 		(at 312.42 120.65)
@@
 		)
 	)
-	(text "RxD"
-		(exclude_from_sim no)
-		(at 359.41 135.89 0)
-		(effects
-			(font
-				(size 1.27 1.27)
-			)
-			(justify left bottom)
-		)
-	)
-	(text "+5V"
-		(exclude_from_sim no)
-		(at 359.41 130.81 0)
-		(effects
-			(font
-				(size 1.27 1.27)
-			)
-			(justify left bottom)
-		)
-	)
-	(text "GND"
-		(exclude_from_sim no)
-		(at 359.41 125.73 0)
-		(effects
-			(font
-				(size 1.27 1.27)
-			)
-			(justify left bottom)
-		)
-	)
-	(text "TxD"
-		(exclude_from_sim no)
-		(at 359.41 133.35 0)
-		(effects
-			(font
-				(size 1.27 1.27)
-			)
-			(justify left bottom)
-		)
-	)
-	(text "CTS"
-		(exclude_from_sim no)
-		(at 359.41 128.27 0)
-		(effects
-			(font
-				(size 1.27 1.27)
-			)
-			(justify left bottom)
-		)
-	)
-	(text "RTS"
-		(exclude_from_sim no)
-		(at 359.41 138.43 0)
-		(effects
-			(font
-				(size 1.27 1.27)
-			)
-			(justify left bottom)
-		)
-	)
 	(label "A13"
 		(at 217.17 250.19 0)
@@
 	(label "A15"
 		(at 328.93 83.82 0)
-		(fields_autoplaced yes)
 		(effects
 			(font
@@
 		)
 	)
+	(embedded_fonts no)
 )
